Commit message: v1

File: series_wheel_legged_robot_ws/install/robot_description_pkg/share/robot_description_pkg/urdf/actor/wheel_link.urdf.xacro (robot description, xacro)
@@ -24,5 +24,5 @@
             <xacro:cylinder_inertia_y m="1.18" r="0.1" h="0.03" xyz="0.0 0.0 0.0" rpy="0.0 0.0 0.0"/>
         </link>
-        <joint name="${position}_wheel_link_joint" type="continuous">
+        <joint name="${position}_wheel_joint" type="continuous">
             <origin xyz="${xyz}" rpy="0.0 0.0 0.0"/>
             <parent link="${position}_shank_link"/>
@@ -30,4 +30,11 @@
             <axis xyz="0.0 1.0 0.0"/>
         </joint>
+         <gazebo reference="${position}_wheel_link">
+	        <material>Gazebo/Yellow</material>
+	        <mu1 value="20.0"/>
+	        <mu2 value="20.0"/>
+	        <kp value="1000000000000000.0"/>
+	        <kd value="1.0"/>
+        </gazebo>
     </xacro:macro>
 </robot>

File: series_wheel_legged_robot_ws/install/robot_description_pkg/share/robot_description_pkg/urdf/base_link.urdf.xacro (robot description, xacro)
@@ -23,5 +23,5 @@
                 </material>
             </collision>
-            <xacro:box_inertia m="3" w="0.2" h="0.3" d="0.2" xyz="0.0 0.0 0.0" rpy="0.0 0.0 0.0"/>
+            <xacro:box_inertia m="3.0" w="0.2" h="0.3" d="0.2" xyz="0.0 0.0 0.0" rpy="0.0 0.0 0.0"/>
         </link>
         <joint name="base_link_joint" type="fixed">
@@ -30,4 +30,7 @@
             <child link="base_link"/>
         </joint>
+        <gazebo reference="base_link">
+	        <material>Gazebo/Green</material>
+        </gazebo>
     </xacro:macro>
 </robot>

File: series_wheel_legged_robot_ws/install/robot_description_pkg/share/robot_description_pkg/urdf/leg_link.urdf.xacro (robot description, xacro)
@@ -45,5 +45,5 @@
             <xacro:box_inertia m="0.135" w="0.025" h="0.02" d="0.3" xyz="0.0 0.0 -0.15" rpy="0.0 0.0 0.0"/>
         </link>
-        <joint name="${position}_thigh_link_joint" type="continuous">
+        <joint name="${position}_hip_joint" type="continuous">
             <origin xyz="${xyz}" rpy="0.0 1.04719755 0.0"/>
             <parent link="base_link"/>
@@ -51,5 +51,5 @@
             <axis xyz="0.0 1.0 0.0"/>
         </joint>
-        <joint name="${position}_shank_link_joint" type="continuous">
+        <joint name="${position}_knee_joint" type="continuous">
             <origin xyz="0.0 0.0 -0.3" rpy="0.0 -2.094395102 0.0"/>
             <parent link="${position}_thigh_link"/>

File: series_wheel_legged_robot_ws/install/robot_description_pkg/share/robot_description_pkg/urdf/series_wheel_legged_robot.urdf.xacro (robot description, xacro)
@@ -8,4 +8,6 @@
 <!-- sensor -->
 <xacro:include filename="$(find robot_description_pkg)/urdf/sensor/imu_link.urdf.xacro"/>
+<!-- ros2_control -->
+<xacro:include filename="$(find robot_description_pkg)/urdf/series_wheel_legged_robot.ros2_control.xacro"/>
 <xacro:base_link_xacro xyz="0.0 0.0 0.6"/>
 <xacro:leg_link_xacro position="left" xyz="0.0 -0.16 -0.07" />
@@ -14,3 +16,4 @@
 <xacro:wheel_link_xacro position="right" xyz="0.0 0.02 -0.3"/>
 <xacro:imu_link_xacro/>
+<xacro:series_wheel_legged_robot_ros2_control/>
 </robot>
